Commit message: first commit

File: urdf/gripper_cross_modal.xacro (robot description, xacro)
@@ -68,3 +68,10 @@
    <child link="sensore"/>
 </joint>
+<link name="finger">
+</link>
+<joint name="finger_joint" type="fixed">
+   <origin xyz="-0.065 -0.035 0.025" rpy="0 0 0"/>
+   <parent link="sensore"/>
+   <child link="finger"/>
+</joint>
 </robot>

Commit message: commit_20_03

File: urdf/gripper_cross_modal.xacro (robot description, xacro)
@@ -71,5 +71,5 @@
 </link>
 <joint name="finger_joint" type="fixed">
-   <origin xyz="-0.065 -0.035 0.025" rpy="0 0 0"/>
+   <origin xyz="-0.065 -0.035 0.025" rpy="1.57079 0 0"/>
    <parent link="sensore"/>
    <child link="finger"/>

Commit message: Esplorazione + PointCloud

File: urdf/gripper_cross_modal.xacro (robot description, xacro)
@@ -75,3 +75,10 @@
    <child link="finger"/>
 </joint>
+<link name="reference_taxel">
+</link>
+<joint name="reference_taxel_joint" type="fixed">
+   <origin xyz="-0.011 -0.005 0.005" rpy="0 0 0"/>
+   <parent link="finger"/>
+   <child link="reference_taxel"/>
+</joint>
 </robot>
